File: KiCad Files/Env-NKL.kicad_pcb (KiCad board)
At the start: 2 copper layers, 366.6 x 119.2 mm, 245 parts, among them J1 TYPE-C-31-M-14, J2 Conn_01x03_Male, SW1 SW_Push, SW2 SW_Push, U1 W25Q16J, U2 3.3V SOT-23-5 5.5V 3.3V, U3 RP2040, Y1 3225_4P

Commit message: named files properly
Connections:
- U3 pad 4: unconnected-(U3-Pad4) -> I2C_SDA
- U3 pad 5: unconnected-(U3-Pad5) -> I2C_SCL
