File: KiCad Files/Env-NKL.kicad_sch (KiCad schematic)
At the start: 247 parts, among them J1 TYPE-C-31-M-14, J2 Conn_01x03_Male, SW1 SW_Push, SW2 SW_Push, U1 W25Q16J, U2 3.3V SOT-23-5 5.5V 3.3V, U3 RP2040, U4 24LC64, Y1 3225_4P

Commit message: named files properly
Parts:
- removed R8, R9: 10K 0402, Resistor_SMD:R_0402_1005Metric, symbol Device:R_Small
- removed U4: 24LC64, Package_SO:SOIC-8_3.9x4.9mm_P1.27mm, symbol Memory_EEPROM:24LC64
Other:
- note removed: "EEPROM for Dynamic Map Storage"

Commit message: changed button footprint so its easier to reset
Parts:
- SW1, SW2: footprint Button_Switch_SMD:SW_Push_SPST_NO_Alps_SKRK -> Button_Switch_SMD:SW_SPST_EVQP7A
Changed lines of the file:
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@@
     (property "Reference" "SW2" (id 0) (at 107.315 327.025 0))
     (property "Value" "SW_Push" (id 1) (at 107.315 329.565 0))
-    (property "Footprint" "Button_Switch_SMD:SW_Push_SPST_NO_Alps_SKRK" (id 2) (at 107.315 329.565 0)
+    (property "Footprint" "Button_Switch_SMD:SW_SPST_EVQP7A" (id 2) (at 107.315 329.565 0)
       (effects (font (size 1.27 1.27)) hide)
     )
@@
     (property "Reference" "SW1" (id 0) (at 27.94 304.165 0))
     (property "Value" "SW_Push" (id 1) (at 27.94 306.705 0))
-    (property "Footprint" "Button_Switch_SMD:SW_Push_SPST_NO_Alps_SKRK" (id 2) (at 27.94 306.705 0)
+    (property "Footprint" "Button_Switch_SMD:SW_SPST_EVQP7A" (id 2) (at 27.94 306.705 0)
       (effects (font (size 1.27 1.27)) hide)
     )
@@
     )
     (path "/fc6b9712-f31f-4f10-8e34-f7d63369a80e"
-      (reference "SW1") (unit 1) (value "SW_Push") (footprint "Button_Switch_SMD:SW_Push_SPST_NO_Alps_SKRK")
+      (reference "SW1") (unit 1) (value "SW_Push") (footprint "Button_Switch_SMD:SW_SPST_EVQP7A")
     )
     (path "/7640aa27-1b5f-487c-9d86-0883b8b27b68"
-      (reference "SW2") (unit 1) (value "SW_Push") (footprint "Button_Switch_SMD:SW_Push_SPST_NO_Alps_SKRK")
+      (reference "SW2") (unit 1) (value "SW_Push") (footprint "Button_Switch_SMD:SW_SPST_EVQP7A")
     )
     (path "/08ea7032-1cdc-4321-96ba-c671c5da2846"

Commit message: improved clearances and fixed issues regarding, made mount holes useable with SMD nuts.
Parts:
- H1, H2, H3, H4, H5, H6, H7: footprint EnvExtras:MountingHole_2.2mm_M2_MODIFIED -> MountingHole:MountingHole_3.7mm_Pad
- Stab1, Stab2, Stab3, Stab4, Stab5, Stab6, Stab7: value MountingHole -> Stabs
Changed lines of the file:
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@@
       (effects (font (size 1.27 1.27)) (justify left))
     )
-    (property "Value" "MountingHole" (id 1) (at 26.67 175.2599 0)
+    (property "Value" "Stabs" (id 1) (at 26.67 175.2599 0)
       (effects (font (size 1.27 1.27)) (justify left) hide)
     )
@@
       (effects (font (size 1.27 1.27)) (justify left))
     )
-    (property "Value" "MountingHole" (id 1) (at 26.67 179.7049 0)
+    (property "Value" "Stabs" (id 1) (at 26.67 179.7049 0)
       (effects (font (size 1.27 1.27)) (justify left) hide)
     )
@@
       (effects (font (size 1.27 1.27)) (justify left) hide)
     )
-    (property "Footprint" "EnvExtras:MountingHole_2.2mm_M2_MODIFIED" (id 2) (at 261.62 278.13 0)
+    (property "Footprint" "MountingHole:MountingHole_3.7mm_Pad" (id 2) (at 261.62 278.13 0)
       (effects (font (size 1.27 1.27)) hide)
     )
@@
       (effects (font (size 1.27 1.27)) (justify left) hide)
     )
-    (property "Footprint" "EnvExtras:MountingHole_2.2mm_M2_MODIFIED" (id 2) (at 274.955 278.13 0)
+    (property "Footprint" "MountingHole:MountingHole_3.7mm_Pad" (id 2) (at 274.955 278.13 0)
       (effects (font (size 1.27 1.27)) hide)
     )
@@
       (effects (font (size 1.27 1.27)) (justify left) hide)
     )
-    (property "Footprint" "EnvExtras:MountingHole_2.2mm_M2_MODIFIED" (id 2) (at 248.285 278.13 0)
+    (property "Footprint" "MountingHole:MountingHole_3.7mm_Pad" (id 2) (at 248.285 278.13 0)
       (effects (font (size 1.27 1.27)) hide)
     )
@@
       (effects (font (size 1.27 1.27)) (justify left))
     )
-    (property "Value" "MountingHole" (id 1) (at 26.67 184.1499 0)
+    (property "Value" "Stabs" (id 1) (at 26.67 184.1499 0)
       (effects (font (size 1.27 1.27)) (justify left) hide)
     )
@@
       (effects (font (size 1.27 1.27)) (justify left))
     )
-    (property "Value" "MountingHole" (id 1) (at 26.67 188.5949 0)
+    (property "Value" "Stabs" (id 1) (at 26.67 188.5949 0)
       (effects (font (size 1.27 1.27)) (justify left) hide)
     )
@@
       (effects (font (size 1.27 1.27)) (justify left) hide)
     )
-    (property "Footprint" "EnvExtras:MountingHole_2.2mm_M2_MODIFIED" (id 2) (at 252.73 278.13 0)
+    (property "Footprint" "MountingHole:MountingHole_3.7mm_Pad" (id 2) (at 252.73 278.13 0)
       (effects (font (size 1.27 1.27)) hide)
     )
@@
       (effects (font (size 1.27 1.27)) (justify left))
     )
-    (property "Value" "MountingHole" (id 1) (at 26.67 193.0399 0)
+    (property "Value" "Stabs" (id 1) (at 26.67 193.0399 0)
       (effects (font (size 1.27 1.27)) (justify left) hide)
     )
@@
       (effects (font (size 1.27 1.27)) (justify left) hide)
     )
-    (property "Footprint" "EnvExtras:MountingHole_2.2mm_M2_MODIFIED" (id 2) (at 266.065 278.13 0)
+    (property "Footprint" "MountingHole:MountingHole_3.7mm_Pad" (id 2) (at 266.065 278.13 0)
       (effects (font (size 1.27 1.27)) hide)
     )
@@
       (effects (font (size 1.27 1.27)) (justify left) hide)
     )
-    (property "Footprint" "EnvExtras:MountingHole_2.2mm_M2_MODIFIED" (id 2) (at 270.51 278.13 0)
+    (property "Footprint" "MountingHole:MountingHole_3.7mm_Pad" (id 2) (at 270.51 278.13 0)
       (effects (font (size 1.27 1.27)) hide)
     )
@@
       (effects (font (size 1.27 1.27)) (justify left) hide)
     )
-    (property "Footprint" "EnvExtras:MountingHole_2.2mm_M2_MODIFIED" (id 2) (at 257.175 278.13 0)
+    (property "Footprint" "MountingHole:MountingHole_3.7mm_Pad" (id 2) (at 257.175 278.13 0)
       (effects (font (size 1.27 1.27)) hide)
     )
@@
       (effects (font (size 1.27 1.27)) (justify left))
     )
-    (property "Value" "MountingHole" (id 1) (at 26.67 201.9299 0)
+    (property "Value" "Stabs" (id 1) (at 26.67 201.9299 0)
       (effects (font (size 1.27 1.27)) (justify left) hide)
     )
@@
       (effects (font (size 1.27 1.27)) (justify left))
     )
-    (property "Value" "MountingHole" (id 1) (at 26.67 197.4849 0)
+    (property "Value" "Stabs" (id 1) (at 26.67 197.4849 0)
       (effects (font (size 1.27 1.27)) (justify left) hide)
     )
@@
     )
     (path "/503f40b7-89aa-48a2-bc09-70062ff13c12"
-      (reference "H1") (unit 1) (value "MountingHole") (footprint "EnvExtras:MountingHole_2.2mm_M2_MODIFIED")
+      (reference "H1") (unit 1) (value "MountingHole") (footprint "MountingHole:MountingHole_3.7mm_Pad")
     )
     (path "/8b39a4c5-9fa4-455e-bbf6-5e1184b9c242"
-      (reference "H2") (unit 1) (value "MountingHole") (footprint "EnvExtras:MountingHole_2.2mm_M2_MODIFIED")
+      (reference "H2") (unit 1) (value "MountingHole") (footprint "MountingHole:MountingHole_3.7mm_Pad")
     )
     (path "/d7ddbfcc-9055-4488-bc82-f181e9834c84"
-      (reference "H3") (unit 1) (value "MountingHole") (footprint "EnvExtras:MountingHole_2.2mm_M2_MODIFIED")
+      (reference "H3") (unit 1) (value "MountingHole") (footprint "MountingHole:MountingHole_3.7mm_Pad")
     )
     (path "/1ae21bad-c702-4a66-9acd-46ae910062e4"
-      (reference "H4") (unit 1) (value "MountingHole") (footprint "EnvExtras:MountingHole_2.2mm_M2_MODIFIED")
+      (reference "H4") (unit 1) (value "MountingHole") (footprint "MountingHole:MountingHole_3.7mm_Pad")
     )
     (path "/a684448d-5397-416b-b9cc-d483dc30d802"
-      (reference "H5") (unit 1) (value "MountingHole") (footprint "EnvExtras:MountingHole_2.2mm_M2_MODIFIED")
+      (reference "H5") (unit 1) (value "MountingHole") (footprint "MountingHole:MountingHole_3.7mm_Pad")
     )
     (path "/b5d704c9-55db-47f8-81a2-4441a8ad91ef"
-      (reference "H6") (unit 1) (value "MountingHole") (footprint "EnvExtras:MountingHole_2.2mm_M2_MODIFIED")
+      (reference "H6") (unit 1) (value "MountingHole") (footprint "MountingHole:MountingHole_3.7mm_Pad")
     )
     (path "/1cf4c225-8eda-4dbe-9ff7-d02eef467c64"
-      (reference "H7") (unit 1) (value "MountingHole") (footprint "EnvExtras:MountingHole_2.2mm_M2_MODIFIED")
+      (reference "H7") (unit 1) (value "MountingHole") (footprint "MountingHole:MountingHole_3.7mm_Pad")
     )
     (path "/8dbc6278-30cb-4300-9284-61363b46f8b2"
@@
     )
     (path "/08ea7032-1cdc-4321-96ba-c671c5da2846"
-      (reference "Stab1") (unit 1) (value "MountingHole") (footprint "Mounting_Keyboard_Stabilizer:Stabilizer_Cherry_MX_2u")
+      (reference "Stab1") (unit 1) (value "Stabs") (footprint "Mounting_Keyboard_Stabilizer:Stabilizer_Cherry_MX_2u")
     )
     (path "/0fc22d86-084e-4672-9047-ba604828e1fd"
-      (reference "Stab2") (unit 1) (value "MountingHole") (footprint "Mounting_Keyboard_Stabilizer:Stabilizer_Cherry_MX_2u")
+      (reference "Stab2") (unit 1) (value "Stabs") (footprint "Mounting_Keyboard_Stabilizer:Stabilizer_Cherry_MX_2u")
     )
     (path "/687251d0-9a0d-489b-9b70-f7e723e02d4b"
-      (reference "Stab3") (unit 1) (value "MountingHole") (footprint "Mounting_Keyboard_Stabilizer:Stabilizer_Cherry_MX_2u")
+      (reference "Stab3") (unit 1) (value "Stabs") (footprint "Mounting_Keyboard_Stabilizer:Stabilizer_Cherry_MX_2u")
     )
     (path "/7618964b-1e2c-4aef-bec8-e346dcf5fd4c"
-      (reference "Stab4") (unit 1) (value "MountingHole") (footprint "Mounting_Keyboard_Stabilizer:Stabilizer_Cherry_MX_2u")
+      (reference "Stab4") (unit 1) (value "Stabs") (footprint "Mounting_Keyboard_Stabilizer:Stabilizer_Cherry_MX_2u")
     )
     (path "/928ebf01-f8a3-4ab9-94fa-685e9e169af1"
-      (reference "Stab5") (unit 1) (value "MountingHole") (footprint "Mounting_Keyboard_Stabilizer:Stabilizer_Cherry_MX_2u")
+      (reference "Stab5") (unit 1) (value "Stabs") (footprint "Mounting_Keyboard_Stabilizer:Stabilizer_Cherry_MX_2u")
     )
     (path "/ff4ccd90-d89d-4c2f-afb4-1b5309e6edf5"
-      (reference "Stab6") (unit 1) (value "MountingHole") (footprint "Mounting_Keyboard_Stabilizer:Stabilizer_Cherry_MX_2u")
+      (reference "Stab6") (unit 1) (value "Stabs") (footprint "Mounting_Keyboard_Stabilizer:Stabilizer_Cherry_MX_2u")
     )
     (path "/f3831990-92ad-4fe6-8a0b-12a455377ffc"
-      (reference "Stab7") (unit 1) (value "MountingHole") (footprint "Mounting_Keyboard_Stabilizer:Stabilizer_Cherry_MX_2u")
+      (reference "Stab7") (unit 1) (value "Stabs") (footprint "Mounting_Keyboard_Stabilizer:Stabilizer_Cherry_MX_2u")
     )
     (path "/24ee306a-932e-4201-9200-975feee8fcf8"
