File: KiCad Files/Main PCB/Env-NKL.kicad_sch (KiCad schematic)
At the start: 244 parts, among them J1 TYPE-C-31-M-14, J2 Conn_01x03_Male, SW1 EVQP7C, SW2 EVQP7C, U1 W25Q16J, U2 3.3V SOT-23-5 5.5V 3.3V, U3 RP2040, Y1 3225_4P 12MHz

Commit message: experimenting & some curiosities with KiCad 7
Parts:
- U1: footprint Package_SO:SOIC-8_3.9x4.9mm_P1.27mm -> Package_SON:SON-8-1EP_3x2mm_P0.5mm_EP1.4x1.6mm

Commit message: swapped board to hotswap, added ANSI keys and re-drew all traces, moved MCU and supporting components to accommodate new stabilisers and switches.
Parts:
- added D_47ANSI1: 1N4148W, Diode_SMD:D_SOD-123, symbol Device:D_Small
- added K_47ANSI1, K_47ANSI2, K_68ANSI1: KEYSW, EnvExtras:MXOnly-1U-Hotswap-Modified, symbol MX_Alps_Hybrid:MX-NoLED
- added Stab(ansi)8, Stab(ansi)9: Stabs, Mounting_Keyboard_Stabilizer:Stabilizer_Cherry_MX_2u, symbol Mechanical:MountingHole
- K_0, K_1, K_10, K_11, K_12, K_13, K_14, K_15, K_151, K_16, K_17, K_18, K_19, K_2, K_20, K_21, K_22, K_23, K_24, K_25, K_26, K_27, K_28, K_29, K_3, K_30, K_31, K_32, K_33, K_34, K_35, K_36, K_37, K_38, K_39, K_4, K_40, K_41, K_42, K_43, K_44, K_45, K_46, K_47, K_48, K_49, K_5, K_50, K_51, K_52, K_53, K_54, K_55, K_56, K_57, K_58, K_59, K_6, K_60, K_61, K_62, K_63, K_64, K_65, K_66, K_67, K_68, K_69, K_7, K_70, K_71, K_72, K_73, K_74, K_75, K_76, K_77, K_78, K_79, K_8, K_80, K_81, K_82, K_83, K_84, K_85, K_86, K_87, K_88, K_89, K_9, K_90, K_91, K_92, K_93, K_94, K_95, K_96, K_97: footprint MX_Only:MXOnly-1U-NoLED -> EnvExtras:MXOnly-1U-Hotswap-Modified
- Y1: value 3225_4P 12MHz -> 3225_4P 12MHz
Connections:
- net col0: now also K_68ANSI1.1 (COL)
- net col14: now also K_47ANSI1.1 (COL), K_47ANSI2.1 (COL)
- net row2: now also D_47ANSI1.1 (K)
- net at D_47.2 (A), K_47.2 (ROW): now also K_47ANSI2.2 (ROW)
- net at D_68.2 (A), K_68.2 (ROW): now also K_68ANSI1.2 (ROW)
- new net: D_47ANSI1.2 (A), K_47ANSI1.2 (ROW)
