File: KiCad Files/BackPlate PCB/Env-NKL-Backplate.kicad_pcb (KiCad board)
At the start: 2 copper layers, 366.6 x 119.2 mm, 9 parts

Commit message: checked alignment and updated incorrect silkscreen.
Other:
- board text added: "EnvKB-NKL | Prototype https://github.com/Envious-Data/Env-NKL"
- board text removed: "EnvKB-TKLQF | Prototype https://github.com/envious-data"
